File: top_plate/therick64BASP_top_plate.kicad_pcb (KiCad board)
At the start: 2 copper layers, 313.1 x 75.2 mm, 77 parts, among them U1 HOLE, U10 HOLE, U11 HOLE, U12 HOLE, U13 HOLE, U14 HOLE, U15 HOLE, U16 HOLE, U17 HOLE, U18 HOLE, U19 HOLE, U2 HOLE, U20 HOLE, U21 HOLE, U22 HOLE, U23 HOLE, U24 HOLE, U25 HOLE, U26 HOLE, U27 HOLE, U28 HOLE, U29 HOLE, U3 HOLE, U30 HOLE, U31 HOLE, U32 HOLE, U33 HOLE, U34 HOLE, U35 HOLE, U36 HOLE, U37 HOLE, U38 HOLE, U39 HOLE, U4 HOLE, U40 HOLE, U41 HOLE, U42 HOLE, U43 HOLE, U44 HOLE, U45 HOLE, U46 HOLE, U47 HOLE, U48 HOLE, U49 HOLE, U5 HOLE, U50 HOLE, U51 HOLE, U52 HOLE, U53 HOLE, U54 HOLE, U55 HOLE, U56 HOLE, U57 HOLE, U58 HOLE, U59 HOLE, U6 HOLE, U60 HOLE, U61 HOLE, U62 HOLE, U63 HOLE, U64 HOLE, U65 HOLE, U66 HOLE, U67 HOLE, U7 HOLE, U8 HOLE, U9 HOLE

Commit message: Changed pins to make routing cleaner
Parts:
- moved U66 2.28 mm to (131.1, 80.2)
- moved U65 1.90 mm to (131.1, 99.2)
- moved U67 1.90 mm to (131.1, 61.2)
Other:
- outline, holes or cut-outs redrawn
- board text added: "therick64BASP Rev 1.0"
- board text removed: "therick64BASP_19mm"

Commit message: Remapped ISP Flash, added mounting holes
Parts:
- added H11: MountingHole, random-keyboard-parts:Generic-Mounthole, F.Cu at (150.1, 61.2)
- added H12: MountingHole, random-keyboard-parts:Generic-Mounthole, F.Cu at (150.1, 99.2)
- added H13: MountingHole, random-keyboard-parts:Generic-Mounthole, F.Cu at (283.1, 61.2)
- added H14: MountingHole, random-keyboard-parts:Generic-Mounthole, F.Cu at (207.1, 61.2)
- added H15: MountingHole, random-keyboard-parts:Generic-Mounthole, F.Cu at (283.1, 99.2)
- added H16: MountingHole, random-keyboard-parts:Generic-Mounthole, F.Cu at (207.1, 99.2)
- added H17: MountingHole, random-keyboard-parts:Generic-Mounthole, F.Cu at (340.1, 61.2)
- added H18: MountingHole, random-keyboard-parts:Generic-Mounthole, F.Cu at (340.1, 99.2)
- H1, H10, H2, H3, H4, H5, H6, H7, H8, H9: footprint random-keyboard-parts:plate_hole_4mm_tht -> random-keyboard-parts:Generic-Mounthole
- moved H4 2.03 mm to (302.1, 61.2)
- moved H2 2.03 mm to (188.1, 61.2)
- moved H7 2.03 mm to (65.0, 61.2)
- moved H6 2.03 mm to (340.1, 80.2)
- moved H1 2.03 mm to (150.1, 80.2)
- moved H5 2.03 mm to (302.1, 99.2)
- moved H3 2.03 mm to (188.1, 99.2)
- moved H9 2.03 mm to (65.0, 99.2)
- moved H8 2.03 mm to (102.9, 61.2)
- moved H10 2.03 mm to (102.9, 99.2)

Commit message: Added mounting holes
Parts:
- H1, H10, H11, H12, H13, H14, H15, H16, H17, H18, H2, H3, H4, H5, H6, H7, H8, H9: footprint random-keyboard-parts:Generic-Mounthole -> random-keyboard-parts:plate_hole_4mm_tht
- moved H13 2.03 mm to (283.0, 63.2)
- moved H17 2.03 mm to (340.0, 63.2)
- moved H4 2.03 mm to (302.0, 63.2)
- moved H7 2.03 mm to (64.9, 63.2)
- moved H11 2.03 mm to (150.0, 63.2)
- moved H14 2.03 mm to (207.0, 63.2)
- moved H2 2.03 mm to (188.0, 63.2)
- moved H15 2.03 mm to (283.0, 101.2)
- moved H18 2.03 mm to (340.0, 101.2)
- moved H5 2.03 mm to (302.0, 101.2)
- moved H6 2.03 mm to (340.0, 82.2)
- moved H9 2.03 mm to (64.9, 101.2)
- moved H1 2.03 mm to (150.0, 82.2)
- moved H12 2.03 mm to (150.0, 101.2)
- moved H16 2.03 mm to (207.0, 101.2)
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