File: 02 top_plate/therick48.16SP_top_plate.kicad_pcb (KiCad board)
At the start: 2 copper layers, 309.7 x 75.2 mm, 85 parts, among them U1 HOLE, U10 HOLE, U11 HOLE, U12 HOLE, U13 HOLE, U14 HOLE, U15 HOLE, U16 HOLE, U17 HOLE, U18 HOLE, U19 HOLE, U2 HOLE, U20 HOLE, U21 HOLE, U22 HOLE, U23 HOLE, U24 HOLE, U25 HOLE, U26 HOLE, U27 HOLE, U28 HOLE, U29 HOLE, U3 HOLE, U30 HOLE, U31 HOLE, U32 HOLE, U33 HOLE, U34 HOLE, U35 HOLE, U36 HOLE, U37 HOLE, U38 HOLE, U39 HOLE, U4 HOLE, U40 HOLE, U41 HOLE, U42 HOLE, U43 HOLE, U44 HOLE, U45 HOLE, U46 HOLE, U47 HOLE, U48 HOLE, U49 HOLE, U5 HOLE, U50 HOLE, U51 HOLE, U52 HOLE, U53 HOLE, U54 HOLE, U55 HOLE, U56 HOLE, U57 HOLE, U58 HOLE, U59 HOLE, U6 HOLE, U60 HOLE, U61 HOLE, U62 HOLE, U63 HOLE, U64 HOLE, U65 HOLE, U66 HOLE, U67 HOLE, U7 HOLE, U8 HOLE, U9 HOLE

Commit message: Added breakaway section, added rotary encoder support
Parts:
- added H19: MountingHole, random-keyboard-parts:plate_hole_4mm_tht, F.Cu at (105.6, 101.2)
- added H20: MountingHole, random-keyboard-parts:plate_hole_4mm_tht, F.Cu at (105.6, 63.2)
- added U68: HOLE, acheron_Hardware:MouseBite_IPC7351, F.Cu at (87.0, 80.2)
- added U69: HOLE, acheron_Hardware:MouseBite_IPC7351, F.Cu at (106.0, 80.2)
- added U70: HOLE, acheron_Hardware:MouseBite_IPC7351, F.Cu at (87.0, 99.2)
- added U71: HOLE, acheron_Hardware:MouseBite_IPC7351, F.Cu at (87.0, 61.2)
- moved H8 19.0 mm to (124.6, 63.2)
- moved H10 19.0 mm to (124.6, 101.2)
Other:
- outline, holes or cut-outs redrawn

Commit message: Update Gerbers
Other:
- board text added: "github.com/dierickdie"
Changed lines of the file:
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@@
   (general
     (thickness 1.6)
-    (drawings 71)
+    (drawings 72)
     (tracks 0)
     (zones 0)
@@
     (solder_mask_min_width 0.25)
     (aux_axis_origin 0 0)
-    (visible_elements FFFFFF7F)
+    (visible_elements FFFFEF7F)
     (pcbplotparams
       (layerselection 0x010fc_ffffffff)
@@
     (pad "" np_thru_hole circle (at 0 0 90) (size 0.8 0.8) (drill 0.8) (layers *.Cu *.Mask))
   )
+  (gr_text github.com/dierickdie (at 245.099355 61.179839) (layer B.SilkS)
+    (effects (font (size 1.5 1.5) (thickness 0.2)) (justify mirror))
+  )
   (gr_line (start 52.439991 117.8) (end 82.459662 117.80003) (layer Edge.Cuts) (width 0.05))
