File: 01 PCB/therick48.16SP.kicad_pcb (KiCad board)
At the start: 2 copper layers, 308.9 x 75.8 mm, 181 parts, among them J1 TYPE-C-31-M12_13, J2 AVR-ISP-6_mod, K1 KEYSW, K10 KEYSW, K11 KEYSW, K12 KEYSW, K13 KEYSW, K14 KEYSW, K15 KEYSW, K16 KEYSW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

Commit message: Small aesthetic tweaks
Other:
- board text added: "open hardware"
- board text added: "therick48.16SP Rev 1.1"
- board text removed: "therick48.16SP Rev 1.0"
